Commit message: cleaned up and updated readme Renamed a couple of files for coinsistency

File: assets/h1/h1.urdf (robot description, URDF)
Before this commit: robot h1_description, 25 links, 24 joints
Links:
- removed link imu_link
- added link L_hand_base_link, mass 0.14143; collision mesh filename=package://h1_description/meshes/L_hand_base_link.STL; visual mesh filename=package://h1_description/meshes/L_hand_base_link.STL
- added link L_index_intermediate, mass 0.0045682; collision mesh filename=package://h1_description/meshes/Link16_L.STL; visual mesh filename=package://h1_description/meshes/Link16_L.STL
- added link L_index_proximal, mass 0.0042405; collision mesh filename=package://h1_description/meshes/Link15_L.STL; visual mesh filename=package://h1_description/meshes/Link15_L.STL
- added link L_middle_intermediate, mass 0.0050397; collision mesh filename=package://h1_description/meshes/Link18_L.STL; visual mesh filename=package://h1_description/meshes/Link18_L.STL
- added link L_middle_proximal, mass 0.0042405; collision mesh filename=package://h1_description/meshes/Link17_L.STL; visual mesh filename=package://h1_description/meshes/Link17_L.STL
- added link L_pinky_intermediate, mass 0.0036036; collision mesh filename=package://h1_description/meshes/Link22_L.STL; visual mesh filename=package://h1_description/meshes/Link22_L.STL
- added link L_pinky_proximal, mass 0.0042405; collision mesh filename=package://h1_description/meshes/Link21_L.STL; visual mesh filename=package://h1_description/meshes/Link21_L.STL
- added link L_ring_intermediate, mass 0.0045682; collision mesh filename=package://h1_description/meshes/Link20_L.STL; visual mesh filename=package://h1_description/meshes/Link20_L.STL
- added link L_ring_proximal, mass 0.0042405; collision mesh filename=package://h1_description/meshes/Link19_L.STL; visual mesh filename=package://h1_description/meshes/Link19_L.STL
- added link L_thumb_distal, mass 0.003344; collision mesh filename=package://h1_description/meshes/Link14_L.STL; visual mesh filename=package://h1_description/meshes/Link14_L.STL
- added link L_thumb_intermediate, mass 0.0037844; collision mesh filename=package://h1_description/meshes/Link13_L.STL; visual mesh filename=package://h1_description/meshes/Link13_L.STL
- added link L_thumb_proximal, mass 0.0066101; collision mesh filename=package://h1_description/meshes/Link12_L.STL; visual mesh filename=package://h1_description/meshes/Link12_L.STL
- added link L_thumb_proximal_base, mass 0.0018869; collision mesh filename=package://h1_description/meshes/Link11_L.STL; visual mesh filename=package://h1_description/meshes/Link11_L.STL
- added link R_hand_base_link, mass 0.14143; collision mesh filename=package://h1_description/meshes/R_hand_base_link.STL; visual mesh filename=package://h1_description/meshes/R_hand_base_link.STL
- added link R_index_intermediate, mass 0.0045683; collision mesh filename=package://h1_description/meshes/Link16_R.STL; visual mesh filename=package://h1_description/meshes/Link16_R.STL
- added link R_index_proximal, mass 0.0042403; collision mesh filename=package://h1_description/meshes/Link15_R.STL; visual mesh filename=package://h1_description/meshes/Link15_R.STL
- added link R_middle_intermediate, mass 0.0050396; collision mesh filename=package://h1_description/meshes/Link18_R.STL; visual mesh filename=package://h1_description/meshes/Link18_R.STL
- added link R_middle_proximal, mass 0.0042403; collision mesh filename=package://h1_description/meshes/Link17_R.STL; visual mesh filename=package://h1_description/meshes/Link17_R.STL
- added link R_pinky_intermediate, mass 0.0035996; collision mesh filename=package://h1_description/meshes/Link22_R.STL; visual mesh filename=package://h1_description/meshes/Link22_R.STL
- added link R_pinky_proximal, mass 0.0042403; collision mesh filename=package://h1_description/meshes/Link21_R.STL; visual mesh filename=package://h1_description/meshes/Link21_R.STL
- added link R_ring_intermediate, mass 0.0045683; collision mesh filename=package://h1_description/meshes/Link20_R.STL; visual mesh filename=package://h1_description/meshes/Link20_R.STL
- added link R_ring_proximal, mass 0.0042403; collision mesh filename=package://h1_description/meshes/Link19_R.STL; visual mesh filename=package://h1_description/meshes/Link19_R.STL
- added link R_thumb_distal, mass 0.0033441; collision mesh filename=package://h1_description/meshes/Link14_R.STL; visual mesh filename=package://h1_description/meshes/Link14_R.STL
- added link R_thumb_intermediate, mass 0.0037847; collision mesh filename=package://h1_description/meshes/Link13_R.STL; visual mesh filename=package://h1_description/meshes/Link13_R.STL
- added link R_thumb_proximal, mass 0.0066075; collision mesh filename=package://h1_description/meshes/Link12_R.STL; visual mesh filename=package://h1_description/meshes/Link12_R.STL
- added link R_thumb_proximal_base, mass 0.0018869; collision mesh filename=package://h1_description/meshes/Link11_R.STL; visual mesh filename=package://h1_description/meshes/Link11_R.STL
- added link left_hand_link, mass 0.014; collision mesh filename=package://h1_description/meshes/left_hand_link.STL; visual mesh filename=package://h1_description/meshes/left_hand_link.STL
- added link right_hand_link, mass 0.014; collision mesh filename=package://h1_description/meshes/right_hand_link.STL; visual mesh filename=package://h1_description/meshes/right_hand_link.STL
- link left_ankle_link: mass 0.725 -> 0.474
- link left_elbow_link: mass 0.745 -> 0.723
- link left_hip_pitch_link: mass 4.953 -> 4.152
- link left_hip_roll_link: mass 2.7150 -> 2.232
- link left_hip_yaw_link: mass 2.965 -> 2.244
- link left_knee_link: mass 2.824 -> 1.721
- link left_shoulder_pitch_link: mass 1.142 -> 1.033
- link left_shoulder_roll_link: mass 0.852 -> 0.793
- link left_shoulder_yaw_link: mass 0.862 -> 0.839
- link pelvis: mass 5.983 -> 5.39
- link right_ankle_link: mass 0.725 -> 0.474
- link right_elbow_link: mass 0.745 -> 0.723
- link right_hip_pitch_link: mass 4.953 -> 4.152
- link right_hip_roll_link: mass 2.7150 -> 2.232
- link right_hip_yaw_link: mass 2.965 -> 2.244
- link right_knee_link: mass 2.824 -> 1.721
- link right_shoulder_pitch_link: mass 1.142 -> 1.033
- link right_shoulder_roll_link: mass 0.852 -> 0.793
- link right_shoulder_yaw_link: mass 0.862 -> 0.839
- link torso_link: mass 17.789 -> 21.189
Joints:
- removed joint imu_joint
- added joint L_base_link_joint: type fixed, parent left_hand_link, child L_hand_base_link, origin xyz=0.003 0 0 rpy=0 0 1.5707963267948966192313216916398
- added joint L_index_intermediate_joint: type revolute, parent L_index_proximal, child L_index_intermediate, origin xyz=-0.0024229 -0.032041 -0.001 rpy=0 0 0, axis 0 0 -1, limit lower=0 upper=1.7 effort=1 velocity=0.5, mimic joint=L_index_proximal_joint multiplier=1 offset=0
- added joint L_index_proximal_joint: type revolute, parent L_hand_base_link, child L_index_proximal, origin xyz=0.00028533 -0.13653 0.032268 rpy=-0.034907 0 0, axis 0 0 -1, limit lower=0 upper=1.7 effort=1 velocity=0.5
- added joint L_middle_intermediate_joint: type revolute, parent L_middle_proximal, child L_middle_intermediate, origin xyz=-0.0024229 -0.032041 -0.001 rpy=0 0 0, axis 0 0 -1, limit lower=0 upper=1.7 effort=1 velocity=0.5, mimic joint=L_middle_proximal_joint multiplier=1 offset=0
- added joint L_middle_proximal_joint: type revolute, parent L_hand_base_link, child L_middle_proximal, origin xyz=0.00028533 -0.1371 0.01295 rpy=0 0 0, axis 0 0 -1, limit lower=0 upper=1.7 effort=1 velocity=0.5
- added joint L_pinky_intermediate_joint: type revolute, parent L_pinky_proximal, child L_pinky_intermediate, origin xyz=-0.0024229 -0.032041 -0.001 rpy=0 0 0, axis 0 0 -1, limit lower=0 upper=1.7 effort=1 velocity=0.5, mimic joint=L_pinky_proximal_joint multiplier=1 offset=0
- added joint L_pinky_proximal_joint: type revolute, parent L_hand_base_link, child L_pinky_proximal, origin xyz=0.00028533 -0.13571 -0.025488 rpy=0.10472 0 0, axis 0 0 -1, limit lower=0 upper=1.7 effort=1 velocity=0.5
- added joint L_ring_intermediate_joint: type revolute, parent L_ring_proximal, child L_ring_intermediate, origin xyz=-0.0024229 -0.032041 -0.001 rpy=0 0 0, axis 0 0 -1, limit lower=0 upper=1.7 effort=1 velocity=0.5, mimic joint=L_ring_proximal_joint multiplier=1 offset=0
- added joint L_ring_proximal_joint: type revolute, parent L_hand_base_link, child L_ring_proximal, origin xyz=0.00028533 -0.13691 -0.0062872 rpy=0.05236 0 0, axis 0 0 -1, limit lower=0 upper=1.7 effort=1 velocity=0.5
- added joint L_thumb_distal_joint: type revolute, parent L_thumb_intermediate, child L_thumb_distal, origin xyz=0.020248 -0.010156 -0.0012 rpy=0 0 0, axis 0 0 -1, limit lower=0 upper=1.2 effort=1 velocity=0.5, mimic joint=L_thumb_proximal_pitch_joint multiplier=2.4 offset=0
- added joint L_thumb_intermediate_joint: type revolute, parent L_thumb_proximal, child L_thumb_intermediate, origin xyz=0.04407 -0.034553 -0.0008 rpy=0 0 0, axis 0 0 -1, limit lower=0 upper=0.8 effort=1 velocity=0.5, mimic joint=L_thumb_proximal_pitch_joint multiplier=1.6 offset=0
- added joint L_thumb_proximal_pitch_joint: type revolute, parent L_thumb_proximal_base, child L_thumb_proximal, origin xyz=0.0099867 0.0098242 -0.0089 rpy=-1.5708 0 0.16939, axis 0 0 -1, limit lower=-0.1 upper=0.6 effort=1 velocity=0.5
- added joint L_thumb_proximal_yaw_joint: type revolute, parent L_hand_base_link, child L_thumb_proximal_base, origin xyz=-0.01696 -0.0691 0.02045 rpy=1.5708 0.5689 3.14159265358979, axis 0 0 1, limit lower=-0.1 upper=1.3 effort=1 velocity=0.5
- added joint R_base_link_joint: type fixed, parent right_hand_link, child R_hand_base_link, origin xyz=0.003 0 0 rpy=0 3.1415926535897932384626433832795 -1.5707963267948966192313216916398
- added joint R_index_intermediate_joint: type revolute, parent R_index_proximal, child R_index_intermediate, origin xyz=-0.0026138 0.032026 -0.001 rpy=0 0 0, axis 0 0 1, limit lower=0 upper=1.7 effort=1 velocity=0.5, mimic joint=R_index_proximal_joint multiplier=1 offset=0
- added joint R_index_proximal_joint: type revolute, parent R_hand_base_link, child R_index_proximal, origin xyz=0.00028533 -0.13653 -0.032268 rpy=-3.1067 0 0, axis 0 0 1, limit lower=0 upper=1.7 effort=1 velocity=0.5
- added joint R_middle_intermediate_joint: type revolute, parent R_middle_proximal, child R_middle_intermediate, origin xyz=-0.0024229 0.032041 -0.001 rpy=0 0 0, axis 0 0 1, limit lower=0 upper=1.7 effort=1 velocity=0.5, mimic joint=R_middle_proximal_joint multiplier=1 offset=0
- added joint R_middle_proximal_joint: type revolute, parent R_hand_base_link, child R_middle_proximal, origin xyz=0.00028533 -0.1371 -0.01295 rpy=-3.1416 0 0, axis 0 0 1, limit lower=0 upper=1.7 effort=1 velocity=0.5
- added joint R_pinky_intermediate_joint: type revolute, parent R_pinky_proximal, child R_pinky_intermediate, origin xyz=-0.0024229 0.032041 -0.001 rpy=0 0 0, axis 0 0 1, limit lower=0 upper=1.7 effort=1 velocity=0.5, mimic joint=R_pinky_proximal_joint multiplier=1 offset=0
- added joint R_pinky_proximal_joint: type revolute, parent R_hand_base_link, child R_pinky_proximal, origin xyz=0.00028533 -0.13571 0.025488 rpy=3.0369 0 0, axis 0 0 1, limit lower=0 upper=1.7 effort=1 velocity=0.5
- added joint R_ring_intermediate_joint: type revolute, parent R_ring_proximal, child R_ring_intermediate, origin xyz=-0.0024229 0.032041 -0.001 rpy=0 0 0, axis 0 0 1, limit lower=0 upper=1.7 effort=1 velocity=0.5, mimic joint=R_ring_proximal_joint multiplier=1 offset=0
- added joint R_ring_proximal_joint: type revolute, parent R_hand_base_link, child R_ring_proximal, origin xyz=0.00028533 -0.13691 0.0062872 rpy=3.0892 0 0, axis 0 0 1, limit lower=0 upper=1.7 effort=1 velocity=0.5
- added joint R_thumb_distal_joint: type revolute, parent R_thumb_intermediate, child R_thumb_distal, origin xyz=0.020248 0.010156 -0.0012 rpy=0 0 0, axis 0 0 1, limit lower=0 upper=1.2 effort=1 velocity=0.5, mimic joint=R_thumb_proximal_pitch_joint multiplier=2.4 offset=0
- added joint R_thumb_intermediate_joint: type revolute, parent R_thumb_proximal, child R_thumb_intermediate, origin xyz=0.04407 0.034553 -0.0008 rpy=0 0 0, axis 0 0 1, limit lower=0 upper=0.8 effort=1 velocity=0.5, mimic joint=R_thumb_proximal_pitch_joint multiplier=1.6 offset=0
- added joint R_thumb_proximal_pitch_joint: type revolute, parent R_thumb_proximal_base, child R_thumb_proximal, origin xyz=-0.0088099 0.010892 -0.00925 rpy=-1.5708 0 -0.16939, axis 0 0 1, limit lower=-0.1 upper=0.6 effort=1 velocity=0.5
- added joint R_thumb_proximal_yaw_joint: type revolute, parent R_hand_base_link, child R_thumb_proximal_base, origin xyz=-0.04096 -0.0691 -0.02045 rpy=1.3708 -2.3689 -0.2854, axis 0 0 -1, limit lower=-0.1 upper=1.3 effort=1 velocity=0.5
- added joint left_hand_joint: type revolute, parent left_elbow_link, child left_hand_link, origin xyz=0.2605 0 -0.0185 rpy=0 0 0, axis 1 0 0, limit lower=-3.0543261909900767596164588448551 upper=3.0543261909900767596164588448551 effort=6 velocity=12
- added joint right_hand_joint: type revolute, parent right_elbow_link, child right_hand_link, origin xyz=0.2605 0 -0.0185 rpy=0 0 0, axis 1 0 0, limit lower=-3.0543261909900767596164588448551 upper=3.0543261909900767596164588448551 effort=6 velocity=12
